File: VuMeterBoard.kicad_sch (KiCad schematic)
At the start: 0 parts

Commit message: push file
Parts:
- added C1: 2.2µF, Capacitor_SMD:C_0603_1608Metric, symbol Device:C
- added C2, C6: 100nF, Capacitor_SMD:C_0603_1608Metric, symbol Device:C
- added C3, C4: 22µF, Capacitor_SMD:CP_Elec_6.3x7.7, symbol Device:C_Polarized
- added C5: 10mF, Capacitor_THT:CP_Radial_D18.0mm_P7.50mm, symbol Device:C_Polarized
- added D1, D2: LL4148, Diode_SMD:D_MiniMELF, symbol Diode:LL4148
- added D3: S2M, Diode_SMD:D_SMB, symbol Device:D
- added F002, F003: T4A, Fuse:Fuseholder_Cylinder-5x20mm_Stelvio-Kontek_PTF78_Horizontal_Open, symbol Device:Fuse
- added F006: T1.6A, Fuse:Fuseholder_Cylinder-5x20mm_Stelvio-Kontek_PTF78_Horizontal_Open, symbol Device:Fuse
- added H1, H2, H3, H4: MountingHole_Pad, MountingHole:MountingHole_3.2mm_M3_Pad_Via, symbol Mechanical:MountingHole_Pad
- added J1, J10, J11, J2, J3, J4, J5, J6, J7, J8, J9: Conn_01x01_Pin, Connector_PinHeader_2.54mm:PinHeader_1x01_P2.54mm_Vertical, symbol Connector:Conn_01x01_Pin
- added R1, R5: 10k, Resistor_SMD:R_0603_1608Metric, symbol Device:R
- added R2, R6: 5k, Potentiometer_SMD:Potentiometer_Vishay_TS53YL_Vertical, symbol Device:R_Potentiometer_Trim
- added R3, R7: 82k, Resistor_SMD:R_0603_1608Metric, symbol Device:R
- added R4, R8: 15k, Resistor_SMD:R_0603_1608Metric, symbol Device:R
- added U1: L78L05_SO8, Package_SO:SOIC-8_3.9x4.9mm_P1.27mm, symbol Regulator_Linear:L78L05_SO8
- added U2: LM358, Package_SO:SOIC-8_3.9x4.9mm_P1.27mm, symbol Amplifier_Operational:LM358
Connections:
- new net: D1.1 (K), J11.1 (Pin_1)
- new net: D1.2 (A), R4.2
- new net: C4.1, J7.1 (Pin_1)
- new net: F003.1, J4.1 (Pin_1)
- new net: C4.2, R5.1
- new net: C3.2, R1.1
- new net: R1.2, R2.1, R2.2
- new net: C3.1, J8.1 (Pin_1)
- new net: F006.1, J6.1 (Pin_1)
- new net: F002.1, J2.1 (Pin_1)
- new net: C1.1, C5.1, D3.1 (K), U1.8 (IN)
- new net: R6.3, R7.1, U2.6 (-)
- new net: R7.2, R8.1, U2.7
- new net: R2.3, R3.1, U2.2 (-)
- new net: R5.2, R6.1, R6.2
- new net: F002.2, J1.1 (Pin_1)
- new net: F003.2, J3.1 (Pin_1)
- new net: R3.2, R4.1, U2.1
- new net: D2.2 (A), R8.2
- new net: D2.1 (K), J9.1 (Pin_1)
- new net: D3.2 (A), F006.2, J5.1 (Pin_1)
- new net +5V: C2.1, C6.1, U1.1 (OUT), U2.8 (V+)
- new net GND: C1.2, C2.2, C5.2, C6.2, H1.1, H2.1, H3.1, H4.1, J10.1 (Pin_1), U1.2 (GND), U1.3 (GND), U1.6 (GND), U1.7 (GND), U2.3 (+), U2.4 (V-), U2.5 (+)
Other:
- note added: "L"
- note added: "R"
- title: (none) -> Vu meter board
